Commit message: Add files via upload

File: src/nagare_description/urdf/base.xacro (robot description, xacro)
@@ -12,8 +12,8 @@
     Vehicle's parameters (remember to enter the model parameters below)
   -->
-  <xacro:property name="mass" value="14.58"/>
-  <!-- <xacro:property name="mass" value="100.00"/> -->
+  <!-- <xacro:property name="mass" value="14.58"/> -->
+  <xacro:property name="mass" value="19.00"/>
   <!-- Center of gravity -->
-  <xacro:property name="cog" value="0 0 -0.1"/>
+  <xacro:property name="cog" value="0 0 0.01"/>
   <!-- Fluid density -->
   <xacro:property name="rho" value="1028"/>
@@ -40,7 +40,7 @@
           <mass value="${mass}" />
           <origin xyz="${cog}" rpy="0 0 0"/>
-          <inertia ixx="0.52" ixy="0.00" ixz="0.00"
-                   iyy="0.41" iyz="0.00"
-                   izz="0.51" />
+          <inertia ixx="0.47" ixy="0.00" ixz="0.02"
+                   iyy="0.55" iyz="0.00"
+                   izz="0.55" />
         </inertial>
         <visual>

File: src/nagare_description/urdf/gazebo.xacro (robot description, xacro)
@@ -3,7 +3,7 @@
     <!-- Center of buoyancy -->
     <xacro:property name="nagare_cob" value="0 0 0"/>
-    <xacro:property name="nagare_volume" value="0.0924"/>
-    <xacro:property name="nagare_length" value="0.5"/>
-    <xacro:property name="nagare_width"  value="0.5"/>
+    <xacro:property name="nagare_volume" value="0.0191"/>
+    <xacro:property name="nagare_length" value="0.4"/>
+    <xacro:property name="nagare_width"  value="0.44"/>
     <xacro:property name="nagare_height" value="0.5"/>
     <xacro:macro name="nagare_hydro_model" params="namespace">

File: src/nagare_description/urdf/snippets.xacro (robot description, xacro)
@@ -17,9 +17,9 @@
       </visual>
       <inertial>
-        <mass value="0.1" />
+        <mass value="0.01" />
         <origin xyz="0 0 0" rpy="0 0 0"/>
-        <inertia ixx="0.000000017" ixy="0.0" ixz="0.0"
-               iyy="0.000000017" iyz="0.0"
-               izz="0.000000017" />
+        <inertia ixx="0.000002852" ixy="0.0" ixz="0.0"
+          iyy="0.000002852" iyz="0.0"
+          izz="0.000004154" />
       </inertial>
     </link>
