Commit message: Add files via upload

File: bluerov_description/urdf/base.xacro (robot description, xacro)
@@ -12,5 +12,6 @@
     Vehicle's parameters (remember to enter the model parameters below)
   -->
-  <xacro:property name="mass" value="8.34"/>
+  <!-- <xacro:property name="mass" value="8.34"/> -->
+    <xacro:property name="mass" value="8.38"/>
   <!-- Center of gravity -->
   <xacro:property name="cog" value="0 0 0"/>

File: bluerov_description/urdf/snippets.xacro (robot description, xacro)
@@ -55,6 +55,6 @@
         <clampMin>-300</clampMin>
         <!-- Minimum and maximum thrust force output allowed -->
-        <thrustMin>-100</thrustMin>
-        <thrustMax>100</thrustMax>
+        <thrustMin>-500</thrustMin>
+        <thrustMax>500</thrustMax>
         <!--
         Value from 0 to 1 to set the efficiency of the output thrust force
