Commit message: Add files via upload

File: nagare_description/urdf/actuators.xacro (robot description, xacro)
@@ -2,4 +2,10 @@
 <robot xmlns:xacro="http://www.ros.org/wiki/xacro">
     <!-- Adding the thruster units with the macro created in snippets.xacro -->
+    <!--
+    Important:
+        - The thruster IDs must be given as integers and must be unique to each thruster unit
+        - The thruster pose in the <origin> block is relative to the body's center of mass. Be
+          aware that Gazebo does not use the SNAME convention per default.
+    -->
     <xacro:thruster_macro robot_namespace="${namespace}" thruster_id="0">
         <origin xyz="0.1 0.15015 0.15913" rpy="0 ${-135*d2r} ${90*d2r}" />

File: nagare_description/urdf/base.xacro (robot description, xacro)
@@ -12,8 +12,7 @@
     Vehicle's parameters (remember to enter the model parameters below)
   -->
-  <!-- <xacro:property name="mass" value="14.58"/> -->
-  <xacro:property name="mass" value="18.3875"/>
+  <xacro:property name="mass" value="18.1875"/>
   <!-- Center of gravity -->
-  <xacro:property name="cog" value="0.0 0.0 0.2"/>
+  <xacro:property name="cog" value="0 0 0"/>
   <!-- Fluid density -->
   <xacro:property name="rho" value="1028"/>
@@ -37,10 +36,17 @@
           otherwise your model will become unstable on Gazebo
         -->
+        <!-- <inertial>
+          <mass value="${mass}" />
+          <origin xyz="${cog}" rpy="0 0 0"/>
+          <inertia ixx="0.52" ixy="0.00" ixz="0.00"
+                   iyy="0.42" iyz="0.00"
+                   izz="0.51" />
+        </inertial> -->
         <inertial>
           <mass value="${mass}" />
           <origin xyz="${cog}" rpy="0 0 0"/>
-          <inertia ixx="0.47" ixy="0.00" ixz="0.00"
-                   iyy="0.48" iyz="0.00"
-                   izz="0.45" />
+          <inertia ixx="3.01" ixy="0.00" ixz="0.00"
+                   iyy="2.59" iyz="0.00"
+                   izz="3.25" />
         </inertial>
         <visual>

File: nagare_description/urdf/snippets.xacro (robot description, xacro)
@@ -48,6 +48,6 @@
         <clampMin>-300</clampMin>
         <!-- Minimum and maximum thrust force output allowed -->
-        <thrustMin>-100</thrustMin>
-        <thrustMax>100</thrustMax>
+        <thrustMin>-500</thrustMin>
+        <thrustMax>500</thrustMax>
         <!--
         Value from 0 to 1 to set the efficiency of the output thrust force
